Commit message: Pipeline working

File: khrylib/assets/mujoco_models/rfc_model/humanoid_root.urdf (robot description, URDF)
Before this commit: robot humanoid, 41 links, 40 joints
Links:
- removed link link1_10
- removed link link1_20
- removed link link1_21
- removed link link1_9
- link lclavicle: mass 0.73651 -> 0.6953470866192378
- link lfemur: mass 3.50634 -> 3.359091094590227
- link lfoot: geometry collision sphere radius=0.08; visual sphere radius=0.08
- link lhumerus: mass 0.86718 -> 0.8359806325536322
- link lradius: mass 0.41397 -> 0.3976078202199582
- link ltibia: mass 1.77925 -> 1.726211085013987
- link lwrist: mass 0.26808 -> 0.26808257310632905
- link rclavicle: mass 0.73651 -> 0.6953470866192378
- link rfemur: mass 3.50634 -> 3.359091094590227
- link rfoot: geometry collision sphere radius=0.08; visual sphere radius=0.08
- link rhumerus: mass 0.86718 -> 0.8359806325536322
- link rradius: mass 0.41397 -> 0.3976078202199582
- link rtibia: mass 1.77925 -> 1.726211085013987
Joints:
- removed joint lfoot_x
- removed joint lfoot_y
- removed joint lfoot_z
- removed joint rfoot_x
- removed joint rfoot_y
- removed joint rfoot_z
- added joint lfoot_fixed: type fixed, parent ltibia, child lfoot, origin xyz=0.13830 0.00000 -0.38000 rpy=0.00000 -0.00000 0.00000, axis -0.34200 0.00000 0.93970
- added joint rfoot_fixed: type fixed, parent rtibia, child rfoot, origin xyz=-0.13830 0.00000 -0.38000 rpy=0.00000 -0.00000 0.00000, axis 0.34200 0.00000 0.93970

Commit message: Add full support of MoE training match performance of nimble with mujoco simulator

File: khrylib/assets/mujoco_models/rfc_model/humanoid_root.urdf (robot description, URDF)
Before this commit: robot humanoid, 37 links, 36 joints
Links:
- added link aux_pitch, mass 0.0
- added link aux_roll, mass 0.0
- added link aux_x, mass 0.0
- added link aux_y, mass 0.0
- added link aux_yaw, mass 0.0
- added link world
- link lfemur: mass 3.359091094590227 -> 3.35909109
- link lfoot: mass 1.23264 -> 2.14466058
- link ltibia: mass 1.726211085013987 -> 1.72621109
- link rfemur: mass 3.359091094590227 -> 3.35909109
- link rfoot: mass 1.23264 -> 2.14466058
- link root: mass 5.57528 -> 5.57527976
- link rtibia: mass 1.726211085013987 -> 1.72621109
- link thorax: mass 4.18879 -> 4.1887902
- link upperback: mass 1.43676 -> 1.43675504
Joints:
- added joint root_pitch: type prismatic, parent world, child aux_pitch, origin xyz=0.00000 0.00000 0.00000 rpy=0.00000 -0.00000 0.00000, axis 1.0 0.0 0.0, limit lower=-100 upper=100 effort=0 velocity=100.0
- added joint root_roll: type prismatic, parent aux_pitch, child aux_roll, origin xyz=0.00000 0.00000 0.00000 rpy=0.00000 -0.00000 0.00000, axis 0.0 1.0 0.0, limit lower=-100 upper=100 effort=0 velocity=100.0
- added joint root_x: type revolute, parent aux_yaw, child aux_x, origin xyz=0.00000 0.00000 0.00000 rpy=0.00000 -0.00000 0.00000, axis 1.0 0.0 0.0, limit lower=-100 upper=100 effort=0 velocity=100.0
- added joint root_y: type revolute, parent aux_x, child aux_y, origin xyz=0.00000 0.00000 0.00000 rpy=0.00000 -0.00000 0.00000, axis 0.0 1.0 0.0, limit lower=-100 upper=100 effort=0 velocity=100.0
- added joint root_yaw: type prismatic, parent aux_roll, child aux_yaw, origin xyz=0.00000 0.00000 0.00000 rpy=0.00000 -0.00000 0.00000, axis 0.0 0.0 1.0, limit lower=-100 upper=100 effort=0 velocity=100.0
- added joint root_z: type revolute, parent aux_y, child root, origin xyz=0.00000 0.00000 0.00000 rpy=0.00000 -0.00000 0.00000, axis 0.0 0.0 1.0, limit lower=-100 upper=100 effort=0 velocity=100.0

Commit message: remove nimble dep

File: khrylib/assets/mujoco_models/rfc_model/humanoid_root.urdf (robot description, URDF)
Before this commit: robot humanoid, 43 links, 42 joints
Links:
- added link link1_10, mass 0.001
- added link link1_20, mass 0.001
- added link link1_21, mass 0.001
- added link link1_9, mass 0.001
- link lfoot: geometry collision box size=0.12000 0.21400 0.04800; visual box size=0.12000 0.21400 0.04800
- link rfoot: geometry collision box size=0.12000 0.21400 0.04800; visual box size=0.12000 0.21400 0.04800
Joints:
- removed joint lfoot_fixed
- removed joint rfoot_fixed
- added joint lfoot_x: type revolute, parent link1_10, child lfoot, origin xyz=0.00000 0.00000 0.00000 rpy=0.00000 -0.00000 0.00000, axis 0.93970 0.00000 0.34200, limit lower=-0.785 upper=1.57 effort=0 velocity=100.0
- added joint lfoot_y: type revolute, parent link1_9, child link1_10, origin xyz=0.00000 0.00000 0.00000 rpy=0.00000 -0.00000 0.00000, axis 0.00000 -1.00000 0.00000, limit lower=-0.785 upper=0.785 effort=0 velocity=100.0
- added joint lfoot_z: type revolute, parent ltibia, child link1_9, origin xyz=0.13830 0.00000 -0.38000 rpy=0.00000 -0.00000 0.00000, axis -0.34200 0.00000 0.93970, limit lower=-0.349 upper=1.22 effort=0 velocity=100.0
- added joint rfoot_x: type revolute, parent link1_21, child rfoot, origin xyz=0.00000 0.00000 0.00000 rpy=0.00000 -0.00000 0.00000, axis 0.93970 0.00000 -0.34200, limit lower=-0.785 upper=1.57 effort=0 velocity=100.0
- added joint rfoot_y: type revolute, parent link1_20, child link1_21, origin xyz=0.00000 0.00000 0.00000 rpy=0.00000 -0.00000 0.00000, axis 0.00000 -1.00000 0.00000, limit lower=-0.785 upper=0.785 effort=0 velocity=100.0
- added joint rfoot_z: type revolute, parent rtibia, child link1_20, origin xyz=-0.13830 0.00000 -0.38000 rpy=0.00000 -0.00000 0.00000, axis 0.34200 0.00000 0.93970, limit lower=-0.349 upper=1.22 effort=0 velocity=100.0
